File: planty1.brd (EAGLE design)
At the start: 115 x 80 mm, 69 parts, among them IC1 LM2596S, IC2 LM2596S, IC3 LM2596S, J2 POWER_JACK, J3 USB_A_SMT_FEMALE, J4 USB_A_SMT_FEMALE, J5 USB_A_SMT_FEMALE, Q1 35A/25V/8.5mΩ, Q2 35A/25V/8.5mΩ, Q3 35A/25V/8.5mΩ

Commit message: schematic cleanup
Parts:
- added FRAME1: FRAME-LEDGERNO_FOOTPRINT, SparkFun-Aesthetics:DUMMY
- C12, C16, C17, C22, C4, C7: value (none) -> 100nF
- R1, R2, R3: value (none) -> 10k
- U$8: value CDRH127 -> CDRH127 - 33uH
Changed lines of the file:
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@@
 </layers>
 <board>
-<fusionsync huburn="a.cGVyc29uYWw6dWUyYmNiYzk5" projecturn="a.cGVyc29uYWw6dWUyYmNiYzk5IzIwMTcwMjAxNjE0NTIyMjY" f3durn="urn:adsk.wipprod:dm.lineage:P6LJSsdnTMS0UlTyof3aIg" pcbguid="9d2a9367-cb74-4049-92d1-8354efb4cba3" lastpulledtime="" lastsyncedchangeguid="" latestrevisionid="4b903c35-988d-4b50-976e-fbbd41b9f6d4" lastsyncedrevisionid="4b903c35-988d-4b50-976e-fbbd41b9f6d4" lastboardhashguid="365ee5b1-b4ea-8c86-af8f-a6831b5e4964" lastpushedtime="2025-05-02T15:31:11Z" linktopcb3d="true"/>
+<fusionsync huburn="a.cGVyc29uYWw6dWUyYmNiYzk5" projecturn="a.cGVyc29uYWw6dWUyYmNiYzk5IzIwMTcwMjAxNjE0NTIyMjY" f3durn="urn:adsk.wipprod:dm.lineage:P6LJSsdnTMS0UlTyof3aIg" pcbguid="" lastpulledtime="" lastsyncedchangeguid="" latestrevisionid="4b903c35-988d-4b50-976e-fbbd41b9f6d4" lastsyncedrevisionid="4b903c35-988d-4b50-976e-fbbd41b9f6d4" lastboardhashguid="365ee5b1-b4ea-8c86-af8f-a6831b5e4964" lastpushedtime="2025-05-02T15:31:11Z" linktopcb3d="false"/>
 <plain>
 <wire x1="0" y1="77" x2="0" y2="3" width="0" layer="20"/>
@@
 <attribute name="VALUE" x="84" y="24.429" size="0.6096" layer="27" font="vector" ratio="20" rot="R180" align="top-center"/>
 </element>
-<element name="C12" library="SparkFun-Capacitors" package="1206" value="" x="84" y="9" smashed="yes" rot="MR180">
+<element name="C12" library="SparkFun-Capacitors" package="1206" value="100nF" x="84" y="9" smashed="yes" rot="MR180">
 <attribute name="NAME" x="84" y="7.857" size="0.6096" layer="26" font="vector" ratio="20" rot="MR180" align="bottom-center"/>
 <attribute name="VALUE" x="84" y="10.143" size="0.6096" layer="28" font="vector" ratio="20" rot="MR180" align="top-center"/>
@@
 <attribute name="VALUE" x="67" y="24.429" size="0.6096" layer="27" font="vector" ratio="20" rot="R180" align="top-center"/>
 </element>
-<element name="C16" library="SparkFun-Capacitors" package="1206" value="" x="67" y="9" smashed="yes" rot="MR180">
+<element name="C16" library="SparkFun-Capacitors" package="1206" value="100nF" x="67" y="9" smashed="yes" rot="MR180">
 <attribute name="NAME" x="67" y="7.857" size="0.6096" layer="26" font="vector" ratio="20" rot="MR180" align="bottom-center"/>
 <attribute name="VALUE" x="67" y="10.143" size="0.6096" layer="28" font="vector" ratio="20" rot="MR180" align="top-center"/>
 </element>
-<element name="C17" library="SparkFun-Capacitors" package="0603" value="" x="24.2" y="40.3" smashed="yes" rot="MR180">
+<element name="C17" library="SparkFun-Capacitors" package="0603" value="100nF" x="24.2" y="40.3" smashed="yes" rot="MR180">
 <attribute name="NAME" x="24.2" y="39.538" size="0.6096" layer="26" font="vector" ratio="20" rot="MR180" align="bottom-center"/>
 <attribute name="VALUE" x="24.2" y="41.062" size="0.6096" layer="28" font="vector" ratio="20" rot="MR180" align="top-center"/>
@@
 <attribute name="VALUE" x="11.01" y="45.361" size="0.6096" layer="27" font="vector" ratio="20" align="top-center"/>
 </element>
-<element name="C22" library="SparkFun-Capacitors" package="1206" value="" x="11" y="42" smashed="yes" rot="MR0">
+<element name="C22" library="SparkFun-Capacitors" package="1206" value="100nF" x="11" y="42" smashed="yes" rot="MR0">
 <attribute name="NAME" x="11" y="43.143" size="0.6096" layer="26" font="vector" ratio="20" rot="MR0" align="bottom-center"/>
 <attribute name="VALUE" x="11" y="40.857" size="0.6096" layer="28" font="vector" ratio="20" rot="MR0" align="top-center"/>
 </element>
-<element name="C4" library="SparkFun-Capacitors" package="1206" value="" x="101" y="9" smashed="yes" rot="MR180">
+<element name="C4" library="SparkFun-Capacitors" package="1206" value="100nF" x="101" y="9" smashed="yes" rot="MR180">
 <attribute name="NAME" x="101" y="7.857" size="0.6096" layer="26" font="vector" ratio="20" rot="MR180" align="bottom-center"/>
 <attribute name="VALUE" x="101" y="10.143" size="0.6096" layer="28" font="vector" ratio="20" rot="MR180" align="top-center"/>
@@
 <attribute name="VALUE" x="11" y="13.571" size="0.6096" layer="27" font="vector" ratio="20" align="top-center"/>
 </element>
-<element name="C7" library="SparkFun-Capacitors" package="1206" value="" x="11" y="22" smashed="yes" rot="MR0">
+<element name="C7" library="SparkFun-Capacitors" package="1206" value="100nF" x="11" y="22" smashed="yes" rot="MR0">
 <attribute name="NAME" x="11" y="23.143" size="0.6096" layer="26" font="vector" ratio="20" rot="MR0" align="bottom-center"/>
 <attribute name="VALUE" x="11" y="20.857" size="0.6096" layer="28" font="vector" ratio="20" rot="MR0" align="top-center"/>
@@
 <attribute name="VALUE" x="50.19" y="16" size="0.6096" layer="27" font="vector" ratio="20" rot="R270" align="top-center"/>
 </element>
-<element name="R1" library="SparkFun-Resistors" package="0603" value=" " x="5" y="53" smashed="yes" rot="MR0">
+<element name="R1" library="SparkFun-Resistors" package="0603" value="10k" x="5" y="53" smashed="yes" rot="MR0">
 <attribute name="NAME" x="5" y="54.143" size="0.6096" layer="26" font="vector" ratio="20" rot="MR0" align="bottom-center"/>
 <attribute name="PROD_ID" value=" " x="-28.02" y="-51.14" size="1.778" layer="28" rot="MR0" display="off"/>
@@
 <attribute name="VALUE" x="30" y="68.238" size="0.6096" layer="27" font="vector" ratio="20" align="top-center"/>
 </element>
-<element name="R2" library="SparkFun-Resistors" package="0603" value=" " x="5" y="51" smashed="yes" rot="MR0">
+<element name="R2" library="SparkFun-Resistors" package="0603" value="10k" x="5" y="51" smashed="yes" rot="MR0">
 <attribute name="NAME" x="5" y="52.143" size="0.6096" layer="26" font="vector" ratio="20" rot="MR0" align="bottom-center"/>
 <attribute name="PROD_ID" value=" " x="-33.1" y="-53.14" size="1.778" layer="28" rot="MR0" display="off"/>
 <attribute name="VALUE" x="5" y="49.857" size="0.6096" layer="28" font="vector" ratio="20" rot="MR0" align="top-center"/>
 </element>
-<element name="R3" library="SparkFun-Resistors" package="0603" value=" " x="5" y="49" smashed="yes" rot="MR0">
+<element name="R3" library="SparkFun-Resistors" package="0603" value="10k" x="5" y="49" smashed="yes" rot="MR0">
 <attribute name="NAME" x="5" y="50.143" size="0.6096" layer="26" font="vector" ratio="20" rot="MR0" align="bottom-center"/>
 <attribute name="PROD_ID" value=" " x="-38.18" y="-55.14" size="1.778" layer="28" rot="MR0" display="off"/>
@@
 <element name="U$6" library="Hatch Prototype" package="CDRH127" value="CDRH127" x="84" y="32" smashed="yes"/>
 <element name="U$7" library="Hatch Prototype" package="SS54" value="SS54" x="92" y="32" smashed="yes" rot="R90"/>
-<element name="U$8" library="Hatch Prototype" package="CDRH127" value="CDRH127" x="67" y="32" smashed="yes"/>
+<element name="U$8" library="Hatch Prototype" package="CDRH127" value="CDRH127 - 33uH" x="67" y="32" smashed="yes"/>
 <element name="U$9" library="Hatch Prototype" package="SS54" value="SS54" x="75" y="32" smashed="yes" rot="R90"/>
 <element name="U1" library="SparkFun-IC-Power" package="SOT223" value="" x="15" y="36.3" smashed="yes" rot="MR90">
@@
 <attribute name="VALUE" x="14.8095" y="35.2205" size="0.4064" layer="28" rot="MR90"/>
 </element>
+<element name="FRAME1" library="SparkFun-Aesthetics" package="DUMMY" value="FRAME-LEDGERNO_FOOTPRINT" x="-23.1" y="-4.1" smashed="yes"/>
 </elements>
 <signals>
