File: planty1.sch (EAGLE design)
At the start: 69 parts, among them IC1 LM2596S, IC2 LM2596S, IC3 LM2596S, J2 POWER_JACK, J3 USB_A_SMT_FEMALE, J4 USB_A_SMT_FEMALE, J5 USB_A_SMT_FEMALE, Q1 35A/25V/8.5mΩ, Q2 35A/25V/8.5mΩ, Q3 35A/25V/8.5mΩ

Commit message: schematic cleanup
Parts:
- added FRAME1: FRAME-LEDGERNO_FOOTPRINT, SparkFun-Aesthetics:FRAME-LEDGERNO_FOOTPRINT
- C12, C16, C17, C22, C4, C7: value (none) -> 100nF
- R1, R2, R3: value (none) -> 10k
- U$8: value CDRH127 -> CDRH127 - 33uH
Other:
- note added: "33uH"
- note added: "5V Fixed DC-DC Buck Converter"
- note added: "AMS1117-3.3"
- note added: "ESP32-C3 Super Mini"
- note added: "High Voltage Low-Side Switching Channels"
- note added: "I2C OLED Display"
- note added: "Power Input"
- note added: "Power Input and Regulation"
- note added: "Push Buttons Debounce"
- note added: "RS485"
- note added: "SS54"
- note added: "USB Switching Channels"
- moved on the sheet: C10, C12, C14, C16, C17, C18, C19, C2, C20, C21, C22, C4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
